File: RevA/ICE40HX8K-B-EVN_23K640/ICE40HX8K-B-EVN_23K640.kicad_sch (KiCad schematic)
At the start: 9 parts

Commit message: schematic done
Parts:
- removed J?: 2x20_Socket, symbol 23K640:2x20_Socket
- added C0, C1, C2, C3, C4, C5, C6, C7, C9: CAP_100nF_0603_6V3, symbol 23K640:CAP_100nF_0603_6V3
- added C8: CAP_4.7uF_0603_6V3, symbol 23K640:CAP_4.7uF_0603_6V3
- added J1: 2x20_Socket, symbol 23K640:2x20_Socket
- gave numbers to parts that had none: 8
Connections:
- net +3V3: now also U4.7 (nHOLD), C0.2, C1.2, C2.2, C3.2, C4.2, C5.2, C6.2, C7.2, C8.2, C9.2, J1.2 (VCCIO)
- net GND: now also C0.1, C1.1, C2.1, C3.1, C4.1, C5.1, C6.1, C8.1, C9.1, J1.15 (GND), J1.16 (GND), J1.23 (GND), J1.24 (GND), J1.31 (GND), J1.32 (GND), J1.39 (GND), J1.40 (GND), J1.7 (GND), J1.8 (GND)
- net nCS_5: now reaches U5.1 (nCS)
- net nCS_5: now also J1.13 (G)
- net S0_5: now reaches U5.2 (SO)
- net S0_5: now also J1.17 (I)
- net SI_5: now reaches U5.5 (SI)
- net SI_5: now also J1.19 (K)
- net at U0.6 (SCK), U1.6 (SCK), U2.6 (SCK)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: now also J1.21 (M)
- net SI_0: now reaches U0.5 (SI)
- net SI_0: now also J1.12 (F)
- net nCS_2: now reaches U2.1 (nCS)
- net nCS_2: now also J1.26 (O)
- net S0_2: now reaches U2.2 (SO)
- net S0_2: now also J1.28 (Q)
- net SI_2: now reaches U2.5 (SI)
- net SI_2: now also J1.30 (S)
- net nCS_3: now reaches U3.1 (nCS)
- net nCS_3: now also J1.34 (U)
- net S0_3: now reaches U3.2 (SO)
- net S0_3: now also J1.36 (W)
- net SI_3: now reaches U3.5 (SI)
- net SI_3: now also J1.38 (Y)
- net nCS_4: now reaches U4.1 (nCS)
- net nCS_4: now also J1.5 (B)
- net S0_4: now reaches U4.2 (SO)
- net S0_4: now also J1.9 (D)
- net nCS_1: now reaches U1.1 (nCS)
- net nCS_1: now also J1.14 (H)
- net S0_0: now reaches U0.2 (SO)
- net S0_0: now also J1.6 (C)
- net S0_1: now reaches U1.2 (SO)
- net S0_1: now also J1.18 (J)
- net nCS_0: now reaches U0.1 (nCS)
- net nCS_0: now also J1.4 (A)
- net SI_1: now reaches U1.5 (SI)
- net SI_1: now also J1.20 (L)
- net nCS_7: now reaches U7.1 (nCS)
- net nCS_7: now also J1.33 (T)
- net S0_7: now reaches U7.2 (SO)
- net S0_7: now also J1.35 (V)
- net SI_7: now reaches U7.5 (SI)
- net SI_7: now also J1.37 (X)
- net nCS_6: now reaches U6.1 (nCS)
- net nCS_6: now also J1.25 (N)
- net S0_6: now reaches U6.2 (SO)
- net S0_6: now also J1.27 (P)
- net SI_6: now reaches U6.5 (SI)
- net SI_6: now also J1.29 (R)
- net SI_4: now reaches U4.5 (SI)
- net SI_4: now also J1.11 (E)
- no-connect marks 8 -> 12

Commit message: footprints
Parts:
- C0, C1, C2, C3, C4, C5, C6, C7, C8, C9: footprint (none) -> 23K640:0603
- J1: footprint (none) -> 23K640:2x20_Header
- U0, U1, U2, U3, U4, U5, U6, U7: footprint (none) -> 23K640:23K640

Commit message: routin
Connections:
- net GND: now also C7.1
- net SI_6: now also J1.25 (N); no longer J1.29 (R)
- net SI_7: now also J1.33 (T); no longer J1.37 (X)
- net nCS_6: now also J1.29 (R); no longer J1.25 (N)
- net nCS_7: now also J1.37 (X); no longer J1.33 (T)
Changed lines of the file:
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@@
+    (stroke (width 0) (type default) (color 0 0 0 0))
+  )
+  (wire (pts (xy 278.13 45.72) (xy 278.13 46.99))
     (stroke (width 0) (type default) (color 0 0 0 0))
   )
@@
     (effects (font (size 1.27 1.27)) (justify left bottom))
   )
-  (label "nCS_6" (at 168.91 133.35 0)
+  (label "nCS_6" (at 168.91 138.43 0)
     (effects (font (size 1.27 1.27)) (justify left bottom))
   )
@@
     (effects (font (size 1.27 1.27)) (justify left bottom))
   )
-  (label "SI_7" (at 168.91 148.59 0)
+  (label "SI_7" (at 168.91 143.51 0)
     (effects (font (size 1.27 1.27)) (justify left bottom))
   )
@@
     (effects (font (size 1.27 1.27)) (justify left bottom))
   )
-  (label "SI_6" (at 168.91 138.43 0)
+  (label "SI_6" (at 168.91 133.35 0)
     (effects (font (size 1.27 1.27)) (justify left bottom))
   )
@@
     (effects (font (size 1.27 1.27)) (justify left bottom))
   )
-  (label "nCS_7" (at 168.91 143.51 0)
-    (effects (font (size 1.27 1.27)) (justify left bottom))
-  )
+  (label "nCS_7" (at 168.91 148.59 0)
+    (effects (font (size 1.27 1.27)) (justify left bottom))
+  )

Commit message: rotate
Connections:
- net SI_0: now also J1.4 (A); no longer J1.12 (F)
- net SI_1: now also J1.14 (H); no longer J1.20 (L)
- net nCS_0: now also J1.12 (F); no longer J1.4 (A)
- net nCS_1: now also J1.20 (L); no longer J1.14 (H)
Changed lines of the file:
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@@
     (effects (font (size 1.27 1.27)) (justify left bottom))
   )
-  (label "SI_1" (at 114.3 125.73 0)
+  (label "SI_1" (at 114.3 118.11 0)
     (effects (font (size 1.27 1.27)) (justify left bottom))
   )
@@
     (effects (font (size 1.27 1.27)) (justify left bottom))
   )
-  (label "nCS_0" (at 114.3 105.41 0)
+  (label "nCS_0" (at 114.3 115.57 0)
     (effects (font (size 1.27 1.27)) (justify left bottom))
   )
@@
     (effects (font (size 1.27 1.27)) (justify left bottom))
   )
-  (label "SI_0" (at 114.3 115.57 0)
+  (label "SI_0" (at 114.3 105.41 0)
     (effects (font (size 1.27 1.27)) (justify left bottom))
   )
@@
     (effects (font (size 1.27 1.27)) (justify left bottom))
   )
-  (label "nCS_1" (at 114.3 118.11 0)
+  (label "nCS_1" (at 114.3 125.73 0)
     (effects (font (size 1.27 1.27)) (justify left bottom))
   )

Commit message: routed
Connections:
- net SI_2: now also J1.26 (O); no longer J1.30 (S)
- net SI_3: now also J1.34 (U); no longer J1.38 (Y)
- net SI_6: now also J1.29 (R); no longer J1.25 (N)
- net SI_7: now also J1.37 (X); no longer J1.33 (T)
- net nCS_2: now also J1.30 (S); no longer J1.26 (O)
- net nCS_3: now also J1.38 (Y); no longer J1.34 (U)
- net nCS_6: now also J1.25 (N); no longer J1.29 (R)
- net nCS_7: now also J1.33 (T); no longer J1.37 (X)
Changed lines of the file:
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@@
     (effects (font (size 1.27 1.27)) (justify left bottom))
   )
-  (label "nCS_6" (at 168.91 138.43 0)
+  (label "nCS_6" (at 168.91 133.35 0)
     (effects (font (size 1.27 1.27)) (justify left bottom))
   )
@@
     (effects (font (size 1.27 1.27)) (justify left bottom))
   )
-  (label "nCS_2" (at 114.3 133.35 0)
+  (label "nCS_2" (at 114.3 138.43 0)
     (effects (font (size 1.27 1.27)) (justify left bottom))
   )
@@
     (effects (font (size 1.27 1.27)) (justify left bottom))
   )
-  (label "SI_7" (at 168.91 143.51 0)
+  (label "SI_7" (at 168.91 148.59 0)
     (effects (font (size 1.27 1.27)) (justify left bottom))
   )
@@
     (effects (font (size 1.27 1.27)) (justify left bottom))
   )
-  (label "SI_6" (at 168.91 133.35 0)
+  (label "SI_6" (at 168.91 138.43 0)
     (effects (font (size 1.27 1.27)) (justify left bottom))
   )
@@
     (effects (font (size 1.27 1.27)) (justify left bottom))
   )
-  (label "SI_3" (at 114.3 148.59 0)
+  (label "SI_3" (at 114.3 143.51 0)
     (effects (font (size 1.27 1.27)) (justify left bottom))
   )
@@
     (effects (font (size 1.27 1.27)) (justify left bottom))
   )
-  (label "SI_2" (at 114.3 138.43 0)
+  (label "SI_2" (at 114.3 133.35 0)
     (effects (font (size 1.27 1.27)) (justify left bottom))
   )
@@
     (effects (font (size 1.27 1.27)) (justify left bottom))
   )
-  (label "nCS_7" (at 168.91 148.59 0)
+  (label "nCS_7" (at 168.91 143.51 0)
     (effects (font (size 1.27 1.27)) (justify left bottom))
   )
@@
     (effects (font (size 1.27 1.27)) (justify left bottom))
   )
-  (label "nCS_3" (at 114.3 143.51 0)
+  (label "nCS_3" (at 114.3 148.59 0)
     (effects (font (size 1.27 1.27)) (justify left bottom))
   )
