File: RevA/ICE40HX8K-B-EVN_23K640/ICE40HX8K-B-EVN_23K640.kicad_pcb (KiCad board)
At the start: 2 copper layers, 19 parts, among them J1 2x20_Socket, U0 23K640, U1 23K640, U2 23K640, U3 23K640, U4 23K640, U5 23K640, U6 23K640, U7 23K640

Commit message: routin
Parts:
- C0, C1, C2, C3, C8, C9, U0, U1, U2, U3: moved to B.Cu
- U4, U5, U6, U7: moved to F.Cu
- moved C9 28.8 mm to (67.4, 119.4), turned to 180 degrees
- moved C8 28.8 mm to (67.4, 116.8), turned to 180 degrees
- moved C0 15.2 mm to (79.9, 116.1), turned to -90 degrees
- moved C3 11.2 mm to (112.9, 116.1), turned to -90 degrees
- moved C4 10.7 mm to (79.5, 112.3), turned to -90 degrees
- moved C2 9.38 mm to (102.8, 116.1), turned to -90 degrees
- moved C7 7.60 mm to (103.3, 118.9), turned to 90 degrees
- moved C6 7.27 mm to (93.1, 118.9), turned to 90 degrees
- moved C1 7.00 mm to (90.0, 116.1)
- moved U5 5.33 mm to (82.4, 113.7), turned to -90 degrees
- moved U4 4.44 mm to (72.2, 113.7), turned to -90 degrees
- moved U3 4.02 mm to (105.2, 117.5), turned to 90 degrees
- moved U0 3.71 mm to (72.2, 117.5), turned to 90 degrees
- moved C5 2.99 mm to (89.8, 115.1), turned to 90 degrees
- moved U7 2.51 mm to (110.7, 117.5), turned to 90 degrees
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Connections:
- C7 pad 1: unconnected-(C7-Pad1) -> GND
- J1 pad 25: /nCS_6 -> /SI_6
- J1 pad 29: /SI_6 -> /nCS_6
- J1 pad 33: /nCS_7 -> /SI_7
- J1 pad 37: /SI_7 -> /nCS_7
Routing:
- net GND: track 0.00 -> 67.8 mm
- net Net-(J1-Pad21): track 0.00 -> 63.5 mm
- net +3V3: track 0.00 -> 31.5 mm
- net /SI_3: track 0.00 -> 14.7 mm
- net /SI_1: track 0.00 -> 14.7 mm
- net /SI_0: track 0.00 -> 14.7 mm
- net /SI_2: track 0.00 -> 14.7 mm
- net /SI_7: track 0.00 -> 13.7 mm
- net /nCS_4: track 0.00 -> 13.3 mm
- net /S0_0: track 0.00 -> 12.9 mm
- net /S0_4: track 0.00 -> 12.4 mm
- net /S0_5: track 0.00 -> 12.2 mm
- net /SI_6: track 0.00 -> 11.9 mm
- net /S0_3: track 0.00 -> 11.1 mm
- net /S0_1: track 0.00 -> 11.1 mm
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- added copper zone on B.Cu, net GND
- added copper zone on F.Cu, net GND
Other:
- board outline added: 50.8 x 16.1 mm

Commit message: rotate
Parts:
- moved C4 10.4 mm to (69.2, 112.8), turned to 0 degrees
- moved U3 5.77 mm to (111.0, 118.3), turned to 180 degrees
- moved U1 4.67 mm to (87.0, 118.3), turned to 180 degrees
- moved U5 4.67 mm to (83.2, 118.3), turned to 0 degrees
- moved U6 4.67 mm to (95.8, 118.3), turned to 0 degrees
- moved U4 4.61 mm to (72.0, 118.3), turned to 0 degrees
- moved U2 4.54 mm to (99.6, 118.3), turned to 180 degrees
- moved U0 3.67 mm to (75.8, 118.3), turned to 180 degrees
- moved C0 3.63 mm to (78.4, 112.8), turned to 180 degrees
- moved U7 3.58 mm to (107.2, 118.3), turned to 0 degrees
- moved C2 2.80 mm to (102.6, 118.9), turned to 90 degrees
- moved C3 2.80 mm to (112.8, 118.9), turned to 90 degrees
- moved C1 2.80 mm to (90.0, 118.9), turned to 90 degrees
Connections:
- J1 pad 12: /SI_0 -> /nCS_0
- J1 pad 14: /nCS_1 -> /SI_1
- J1 pad 20: /SI_1 -> /nCS_1
- J1 pad 4: /nCS_0 -> /SI_0
Routing:
- net GND: track 67.8 -> 0.00 mm
- net Net-(J1-Pad21): track 63.5 -> 0.00 mm
- net /SI_3: track 14.7 -> 0.00 mm
- net /SI_2: track 14.7 -> 0.00 mm
- net /SI_7: track 13.7 -> 0.00 mm
- net /S0_5: track 12.2 -> 0.00 mm
- net /SI_6: track 11.9 -> 0.00 mm
- net /S0_3: track 11.1 -> 0.00 mm
- net /S0_2: track 11.1 -> 0.00 mm
- net /S0_6: track 11.0 -> 0.00 mm
- net /S0_7: track 9.32 -> 0.00 mm
- net /nCS_7: track 7.73 -> 0.00 mm
- net /nCS_3: track 7.58 -> 0.00 mm
- net /nCS_2: track 7.58 -> 0.00 mm
- net /nCS_6: track 7.49 -> 0.00 mm
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Other:
- board size 50.8 x 16.1 mm -> 50.8 x 17.4 mm

Commit message: routed
Parts:
- moved C5 9.65 mm to (80.4, 112.9), turned to 0 degrees
- moved C7 6.17 mm to (104.5, 112.9), turned to 0 degrees
- moved C3 6.05 mm to (113.7, 112.9), turned to 180 degrees
- moved C2 6.01 mm to (102.2, 112.9), turned to 180 degrees
- moved C1 5.98 mm to (89.7, 112.9), turned to 180 degrees
- moved C6 5.97 mm to (93.0, 112.9), turned to 0 degrees
- moved C8 0.51 mm to (67.9, 116.8)
- moved C9 0.51 mm to (67.9, 119.4)
- moved C4 0.23 mm to (69.3, 112.9)
- moved C0 0.18 mm to (78.5, 112.9)
Connections:
- J1 pad 25: /SI_6 -> /nCS_6
- J1 pad 26: /nCS_2 -> /SI_2
- J1 pad 29: /nCS_6 -> /SI_6
- J1 pad 30: /SI_2 -> /nCS_2
- J1 pad 33: /SI_7 -> /nCS_7
- J1 pad 34: /nCS_3 -> /SI_3
- J1 pad 37: /nCS_7 -> /SI_7
- J1 pad 38: /SI_3 -> /nCS_3
Routing:
- net +3V3: track 30.0 -> 190.2 mm, vias 2 -> 79
- net GND: track 0.00 -> 73.5 mm, vias 0 -> 67
- net Net-(J1-Pad21): track 0.00 -> 62.4 mm, vias 0 -> 4
- net /SI_2: track 0.00 -> 15.8 mm
- net /SI_3: track 0.00 -> 14.0 mm
- net /SI_7: track 0.00 -> 13.2 mm
- net /SI_6: track 0.00 -> 12.4 mm
- net /SI_5: track 0.00 -> 12.4 mm
- net /nCS_2: track 0.00 -> 7.48 mm
- net /S0_6: track 0.00 -> 7.02 mm
- net /nCS_5: track 0.00 -> 6.98 mm
- net /S0_5: track 0.00 -> 6.98 mm
- net /nCS_3: track 0.00 -> 6.52 mm
- net /S0_7: track 0.00 -> 6.52 mm
- net /S0_2: track 0.00 -> 6.51 mm
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- added copper zone on B.Cu, net +3V3
- added copper zone on F.Cu, net +3V3

Commit message: pcb
Routing:
- net +3V3: vias 79 -> 76

Commit message: added fab output
Routing:
- net +3V3: track 190.2 -> 196.8 mm, vias 76 -> 65
- net GND: track 73.5 -> 70.2 mm, vias 67 -> 65
- net /SI_2: track 15.8 -> 15.0 mm
Other:
- board text added: "23K640 SRAM"
- board text added: "AJR RevA March 2023"
